File: Kicad/PicoPAC.kicad_sch (KiCad schematic)
At the start: 5 parts, among them J1 Videopac-edgeconnector, J2 Conn_01x20, J3 Conn_01x20, SW1 SW_Push

Commit message: faulty attempt to fix in game reset
Parts:
- added R1: 10k, Resistor_THT:R_Axial_DIN0207_L6.3mm_D2.5mm_P7.62mm_Horizontal, symbol Device:R
- added SW2: SW_Push, Button_Switch_THT:SW_PUSH_6mm, symbol Switch:SW_Push
- D1: value Diode -> Diode
Connections:
- net +3.3V: now reaches J3.4 (Pin_4)
- net +3.3V: now also R1.2
- net RESTART: now reaches J3.9 (Pin_9)
- net RESTART: now also SW2.1
- new net: R1.1, SW2.2
- no-connect marks 6 -> 4
